File: hardware/electronics/joint_controller_board/rev_b/joint_controller_board_rev_b.kicad_pcb (KiCad board)
At the start: 2 copper layers, 72 x 128 mm, 30 parts, among them J1 V_IN_5V, J2 XT60_48V_IN, J3 XT60_48V_OUT, J4 CAN_Servo, J5 CAN_Controller, J6 8P8C, Q1 IRFB4110PBF, Q2 IRFB4110PBF, U1 Pico, U2 LM2576HVT-12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

Commit message: fix(electronics): Correct U4 footprint for TI DCU package (Rev B.3)
U4 (SN74LVC2G08DCUR) footprint was wrong:
- Old: VSSOP-8_3.0x3.0mm_P0.65mm (generic)
- New: VSSOP-8_2.4x2.1mm_P0.5mm (TI DCU/US8)

Issue discovered during PCBWay assembly - component didn't fit pads.
TI's DCU package uses 0.5mm pitch, not 0.65mm.

Updated:
- KiCad schematic and PCB
- Regenerated Gerber files
- BOM and README changelog
Parts:
- F1: value Fuseholder (ATO/ATC) -> 40A
- U4: footprint Package_SO:VSSOP-8_3.0x3.0mm_P0.65mm -> Package_SO:VSSOP-8_2.4x2.1mm_P0.5mm
Routing:
- net GP22: track 70.2 -> 69.4 mm
- net SAFETY_EN: track 29.2 -> 29.8 mm
- net Net-(U_WDT1-~{WDO}): track 71.9 -> 72.6 mm
- net +3V3: track 99.3 -> 98.7 mm
