File: hardware/electronics/joint_controller_board/rev_b/joint_controller_board_rev_b.kicad_sch (KiCad schematic)
At the start: 30 parts, among them J1 V_IN_5V, J2 XT60_48V_IN, J3 XT60_48V_OUT, J4 CAN_Servo, J5 CAN_Controller, J6 8P8C, Q1 IRFB4110PBF, Q2 IRFB4110PBF, U1 Pico, U2 LM2576HVT-12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

Commit message: fix(electronics): Correct U4 footprint for TI DCU package (Rev B.3)
U4 (SN74LVC2G08DCUR) footprint was wrong:
- Old: VSSOP-8_3.0x3.0mm_P0.65mm (generic)
- New: VSSOP-8_2.4x2.1mm_P0.5mm (TI DCU/US8)

Issue discovered during PCBWay assembly - component didn't fit pads.
TI's DCU package uses 0.5mm pitch, not 0.65mm.

Updated:
- KiCad schematic and PCB
- Regenerated Gerber files
- BOM and README changelog
Parts:
- U4: footprint Package_SO:VSSOP-8_3.0x3.0mm_P0.65mm -> Package_SO:VSSOP-8_2.4x2.1mm_P0.5mm
Changed lines of the file:
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@@
       (effects (font (size 1.27 1.27)))
     )
-    (property "Footprint" "Package_SO:VSSOP-8_3.0x3.0mm_P0.65mm" (at 128.27 139.7 0)
+    (property "Footprint" "Package_SO:VSSOP-8_2.4x2.1mm_P0.5mm" (at 128.27 139.7 0)
       (effects (font (size 1.27 1.27)) hide)
     )
@@
       (effects (font (size 1.27 1.27)))
     )
-    (property "Footprint" "Package_SO:VSSOP-8_3.0x3.0mm_P0.65mm" (at 128.27 157.48 0)
+    (property "Footprint" "Package_SO:VSSOP-8_2.4x2.1mm_P0.5mm" (at 128.27 157.48 0)
       (effects (font (size 1.27 1.27)) hide)
     )
@@
       (effects (font (size 1.27 1.27)) (justify left))
     )
-    (property "Footprint" "Package_SO:VSSOP-8_3.0x3.0mm_P0.65mm" (at 125.73 181.61 0)
-      (effects (font (size 1.27 1.27)) hide)
-    )
+    (property "Footprint" "Package_SO:VSSOP-8_2.4x2.1mm_P0.5mm" (at 125.73 181.61 0)
+      (effects (font (size 1.27 1.27)) hide)
+    )
