File: hardware/electronics/joint_controller_board/rev_d_logic/joint_controller_board_rev_d_logic.kicad_pcb (KiCad board)
At the start: 2 copper layers, 40 x 60 mm, 43 parts, among them J1 J_IFACE, J2 J_ENCODERS, U1 Pico, U4 SN74LVC2G08, Y1 8MHz, Y2 8MHz

Commit message: hardware: align rev d logic raw monitor net
Connections:
- net VIN_POST_F1_MON renamed VIN_RAW_MON
Changed lines of the file:
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@@
 	(net 51 "FAULT_N")
 	(net 52 "PWRGD_N")
-	(net 53 "VIN_POST_F1_MON")
+	(net 53 "VIN_RAW_MON")
 	(net 54 "Net-(U_CAN2-OSC2)")
 	(net 55 "Net-(U_CAN2-OSC1)")
@@
 			(layers "*.Cu" "*.Mask")
 			(remove_unused_layers no)
-			(net 53 "VIN_POST_F1_MON")
+			(net 53 "VIN_RAW_MON")
 			(pinfunction "GPIO26_ADC0")
 			(pintype "bidirectional")
@@
 			(layers "*.Cu" "*.Mask")
 			(remove_unused_layers no)
-			(net 53 "VIN_POST_F1_MON")
+			(net 53 "VIN_RAW_MON")
 			(pintype "passive")
 		)
